Commit message: .

File: manipulator/parallel_spherical/parallel_spherical.urdf (robot description, URDF)
Before this commit: robot parallel_spherical, 7 links, 6 joints
Links:
- removed link lower_link31
- added link ring1, mass 0.9575334104776773; collision mesh filename=meshes/ring1.stl scale=0.001 0.001 0.001; visual mesh filename=meshes/ring1.stl scale=0.001 0.001 0.001
- link base_link: mass 0.9575334104776773 -> 0.4147232258009921
- link lower_link21: mass 0.3882295327079039 -> 0.38822953270790367
- link upper_link21: mass 0.3201192652534844 -> 0.3201192652534845
Joints:
- removed joint 1-1
- removed joint 2-2
- removed joint 3-3
- removed joint base-1
- removed joint base-2
- removed joint base-3
- added joint Revolute_60: type continuous, parent base_link, child lower_link21, origin xyz=0.0 0.0 -0.1375 rpy=0 0 0, axis 0.0 0.0 -1.0
- added joint Revolute_61: type continuous, parent lower_link21, child lower_link11, origin xyz=0.0 -0.0 0.015 rpy=0 0 0, axis 0.0 0.0 -1.0
- added joint Revolute_62: type continuous, parent lower_link11, child upper_link11, origin xyz=0.115 0.0 0.13 rpy=0 0 0, axis 1.0 0.0 0.0
- added joint Revolute_63: type continuous, parent lower_link21, child upper_link21, origin xyz=-0.0575 0.099593 0.145 rpy=0 0 0, axis -0.5 0.866025 -0.0
- added joint Revolute_64: type continuous, parent base_link, child upper_link31, origin xyz=-0.0575 -0.099593 0.0075 rpy=0 0 0, axis -0.5 -0.866025 0.0
- added joint Revolute_68: type continuous, parent upper_link11, child ring1, origin xyz=-0.115 0.1 0.0 rpy=0 0 0, axis 0.0 1.0 -0.0
